File: kicad/Didj-Fi.sch (KiCad schematic (older format))
At the start: 20 parts, among them J1 didj_cart, J3 USB_B_Micro, U1 CH340E, U2 ESP-12F

Commit message: prepare for manufacture
Parts:
- C1, C2, C4: LCSC (none) -> C309458
- C3: LCSC (none) -> C45783
- J3: footprint Connector_USB:USB_Micro-B_Molex_47346-0001 -> project:C40942
- R1, R11, R3, R4, R5, R7, R8, R9: LCSC (none) -> C25744
- R10, R2: LCSC (none) -> C25900
- R6: LCSC (none) -> C25784
- U1: LCSC (none) -> C99652
Changed lines of the file:
@@
 F 2 "Capacitor_SMD:C_0805_2012Metric" H 5438 4750 50  0001 C CNN
 F 3 "~" H 5400 4900 50  0001 C CNN
+F 4 "C45783" H 5400 4900 50  0001 C CNN "LCSC"
 	1    5400 4900
 	1    0    0    -1
@@
 F 2 "Capacitor_SMD:C_0402_1005Metric" H 5838 4750 50  0001 C CNN
 F 3 "~" H 5800 4900 50  0001 C CNN
+F 4 "C309458" H 5800 4900 50  0001 C CNN "LCSC"
 	1    5800 4900
 	1    0    0    -1
@@
 F 2 "Capacitor_SMD:C_0402_1005Metric" H 4438 2100 50  0001 C CNN
 F 3 "~" H 4400 2250 50  0001 C CNN
+F 4 "C309458" H 4400 2250 50  0001 C CNN "LCSC"
 	1    4400 2250
 	1    0    0    -1
@@
 F 2 "Resistor_SMD:R_0402_1005Metric" V 4390 4290 50  0001 C CNN
 F 3 "~" H 4350 4300 50  0001 C CNN
+F 4 "C25744" H 4350 4300 50  0001 C CNN "LCSC"
 	1    4350 4300
 	0    1    1    0
@@
 F 2 "Resistor_SMD:R_0402_1005Metric" V 4640 4490 50  0001 C CNN
 F 3 "~" H 4600 4500 50  0001 C CNN
+F 4 "C25744" H 4600 4500 50  0001 C CNN "LCSC"
 	1    4600 4500
 	0    1    1    0
@@
 F 2 "Resistor_SMD:R_0402_1005Metric" V 4640 4890 50  0001 C CNN
 F 3 "~" H 4600 4900 50  0001 C CNN
+F 4 "C25744" H 4600 4900 50  0001 C CNN "LCSC"
 	1    4600 4900
 	0    1    1    0
@@
 F 2 "Resistor_SMD:R_0402_1005Metric" V 4390 4690 50  0001 C CNN
 F 3 "~" H 4350 4700 50  0001 C CNN
+F 4 "C25744" H 4350 4700 50  0001 C CNN "LCSC"
 	1    4350 4700
 	0    1    1    0
@@
 F 2 "Resistor_SMD:R_0402_1005Metric" V 4640 4090 50  0001 C CNN
 F 3 "~" H 4600 4100 50  0001 C CNN
+F 4 "C25784" H 4600 4100 50  0001 C CNN "LCSC"
 	1    4600 4100
 	0    1    1    0
@@
 F 2 "Resistor_SMD:R_0402_1005Metric" V 4390 5090 50  0001 C CNN
 F 3 "~" H 4350 5100 50  0001 C CNN
+F 4 "C25744" H 4350 5100 50  0001 C CNN "LCSC"
 	1    4350 5100
 	0    1    1    0
@@
 F 2 "Resistor_SMD:R_0402_1005Metric" V 4640 5690 50  0001 C CNN
 F 3 "~" H 4600 5700 50  0001 C CNN
+F 4 "C25744" H 4600 5700 50  0001 C CNN "LCSC"
 	1    4600 5700
 	0    1    1    0
@@
 F 2 "Capacitor_SMD:C_0402_1005Metric" H 4788 2100 50  0001 C CNN
 F 3 "~" H 4750 2250 50  0001 C CNN
+F 4 "C309458" H 4750 2250 50  0001 C CNN "LCSC"
 	1    4750 2250
 	1    0    0    -1
@@
 F 2 "Resistor_SMD:R_0402_1005Metric" V 3390 7090 50  0001 C CNN
 F 3 "~" H 3350 7100 50  0001 C CNN
+F 4 "C25900" V 3350 7100 50  0001 C CNN "LCSC"
 	1    3350 7100
 	0    1    1    0
@@
 F 2 "Resistor_SMD:R_0402_1005Metric" V 1890 7090 50  0001 C CNN
 F 3 "~" H 1850 7100 50  0001 C CNN
+F 4 "C25900" V 1850 7100 50  0001 C CNN "LCSC"
 	1    1850 7100
 	0    1    1    0
@@
 F 2 "project:MSOP10" H 6000 2300 50  0001 L BNN
 F 3 "IC-14135" H 6000 2300 50  0001 L BNN
+F 4 "C99652" H 6000 2300 50  0001 C CNN "LCSC"
 	1    6000 2300
 	1    0    0    -1
@@
 F 0 "J3" H 3305 2667 50  0000 C CNN
 F 1 "USB_B_Micro" H 3305 2576 50  0000 C CNN
-F 2 "Connector_USB:USB_Micro-B_Molex_47346-0001" H 3400 2150 50  0001 C CNN
+F 2 "project:C40942" H 3400 2150 50  0001 C CNN
 F 3 "~" H 3400 2150 50  0001 C CNN
 	1    3250 2200
@@
 F 2 "Resistor_SMD:R_0402_1005Metric" V 4340 5490 50  0001 C CNN
 F 3 "~" H 4300 5500 50  0001 C CNN
+F 4 "C25744" H 4300 5500 50  0001 C CNN "LCSC"
 	1    4300 5500
 	0    1    1    0
@@
 F 2 "Resistor_SMD:R_0402_1005Metric" V 4640 5290 50  0001 C CNN
 F 3 "~" H 4600 5300 50  0001 C CNN
+F 4 "C25744" H 4600 5300 50  0001 C CNN "LCSC"
 	1    4600 5300
 	0    1    1    0
