File: kicad/Didj-Fi_NAND.sch (KiCad schematic (older format))
At the start: 23 parts, among them J1 didj_cart, J2 Conn_01x04_Male, U1 NAND-8BIT, U2 ESP-12F

Commit message: prepare for manufacture
Parts:
- C1, C2, C4: LCSC (none) -> C309458
- C3: LCSC (none) -> C45783
- R1, R10, R2: LCSC (none) -> C25900
- R11, R12, R3, R4, R5, R7, R8: LCSC (none) -> C25744
- R6: LCSC (none) -> C25784
- R9: value 4.7k -> 10k; LCSC (none) -> C25744
- U1: LCSC (none) -> C117899
Changed lines of the file:
@@
 F 2 "Capacitor_SMD:C_0805_2012Metric" H 4388 4550 50  0001 C CNN
 F 3 "~" H 4350 4700 50  0001 C CNN
+F 4 "C45783" H 4350 4700 50  0001 C CNN "LCSC"
 	1    4350 4700
 	1    0    0    -1
@@
 F 2 "Capacitor_SMD:C_0402_1005Metric" H 4788 4550 50  0001 C CNN
 F 3 "~" H 4750 4700 50  0001 C CNN
+F 4 "C309458" H 4750 4700 50  0001 C CNN "LCSC"
 	1    4750 4700
 	1    0    0    -1
@@
 F 2 "Capacitor_SMD:C_0402_1005Metric" H 3038 1850 50  0001 C CNN
 F 3 "~" H 3000 2000 50  0001 C CNN
+F 4 "C309458" H 3000 2000 50  0001 C CNN "LCSC"
 	1    3000 2000
 	1    0    0    -1
@@
 F 2 "Resistor_SMD:R_0402_1005Metric" V 3340 4140 50  0001 C CNN
 F 3 "~" H 3300 4150 50  0001 C CNN
+F 4 "C25744" H 3300 4150 50  0001 C CNN "LCSC"
 	1    3300 4150
 	0    1    1    0
@@
 F 2 "Resistor_SMD:R_0402_1005Metric" V 3590 4340 50  0001 C CNN
 F 3 "~" H 3550 4350 50  0001 C CNN
+F 4 "C25744" H 3550 4350 50  0001 C CNN "LCSC"
 	1    3550 4350
 	0    1    1    0
@@
 F 2 "Resistor_SMD:R_0402_1005Metric" V 3590 4740 50  0001 C CNN
 F 3 "~" H 3550 4750 50  0001 C CNN
+F 4 "C25744" H 3550 4750 50  0001 C CNN "LCSC"
 	1    3550 4750
 	0    1    1    0
@@
 F 2 "Resistor_SMD:R_0402_1005Metric" V 3340 4540 50  0001 C CNN
 F 3 "~" H 3300 4550 50  0001 C CNN
+F 4 "C25744" H 3300 4550 50  0001 C CNN "LCSC"
 	1    3300 4550
 	0    1    1    0
@@
 F 2 "Resistor_SMD:R_0402_1005Metric" V 3590 3940 50  0001 C CNN
 F 3 "~" H 3550 3950 50  0001 C CNN
+F 4 "C25784" H 3550 3950 50  0001 C CNN "LCSC"
 	1    3550 3950
 	0    1    1    0
@@
 F 2 "Resistor_SMD:R_0402_1005Metric" V 3340 4940 50  0001 C CNN
 F 3 "~" H 3300 4950 50  0001 C CNN
+F 4 "C25744" H 3300 4950 50  0001 C CNN "LCSC"
 	1    3300 4950
 	0    1    1    0
@@
 P 3550 5550
 F 0 "R9" H 3618 5596 50  0000 L CNN
-F 1 "4.7k" H 3618 5505 50  0000 L CNN
+F 1 "10k" H 3618 5505 50  0000 L CNN
 F 2 "Resistor_SMD:R_0402_1005Metric" V 3590 5540 50  0001 C CNN
 F 3 "~" H 3550 5550 50  0001 C CNN
+F 4 "C25744" H 3550 5550 50  0001 C CNN "LCSC"
 	1    3550 5550
 	0    1    1    0
@@
 F 2 "project:TSOP48" H 4450 2050 50  0001 C CNN
 F 3 "" H 4450 2050 50  0001 C CNN
+F 4 "C117899" H 4450 2050 50  0001 C CNN "LCSC"
 	1    4450 2050
 	1    0    0    -1
@@
 F 2 "Capacitor_SMD:C_0402_1005Metric" H 3388 1850 50  0001 C CNN
 F 3 "~" H 3350 2000 50  0001 C CNN
+F 4 "C309458" H 3350 2000 50  0001 C CNN "LCSC"
 	1    3350 2000
 	1    0    0    -1
@@
 F 2 "Resistor_SMD:R_0402_1005Metric" V 3990 7090 50  0001 C CNN
 F 3 "~" H 3950 7100 50  0001 C CNN
+F 4 "C25900" V 3950 7100 50  0001 C CNN "LCSC"
 	1    3950 7100
 	0    1    1    0
@@
 F 2 "Resistor_SMD:R_0402_1005Metric" V 2940 7090 50  0001 C CNN
 F 3 "~" H 2900 7100 50  0001 C CNN
+F 4 "C25900" V 2900 7100 50  0001 C CNN "LCSC"
 	1    2900 7100
 	0    1    1    0
@@
 F 2 "Resistor_SMD:R_0402_1005Metric" V 1840 7090 50  0001 C CNN
 F 3 "~" H 1800 7100 50  0001 C CNN
+F 4 "C25900" V 1800 7100 50  0001 C CNN "LCSC"
 	1    1800 7100
 	0    1    1    0
@@
 F 2 "Resistor_SMD:R_0402_1005Metric" V 3590 5140 50  0001 C CNN
 F 3 "~" H 3550 5150 50  0001 C CNN
+F 4 "C25744" H 3550 5150 50  0001 C CNN "LCSC"
 	1    3550 5150
 	0    1    1    0
@@
 F 2 "Resistor_SMD:R_0402_1005Metric" V 3340 5340 50  0001 C CNN
 F 3 "~" H 3300 5350 50  0001 C CNN
+F 4 "C25744" H 3300 5350 50  0001 C CNN "LCSC"
 	1    3300 5350
 	0    1    1    0
